Commit message: Update adaptive_gripper.urdf.xacro

File: adaptive_gripper.urdf.xacro (robot description, xacro)
@@ -42,6 +42,6 @@
       </collision>
     </link>
-    <joint name="${parent}_to_gripper_base" type="fixed">
-      <parent link="${parent}"/>
+    <joint name="$link6_flange_to_gripper_base" type="fixed">
+      <parent link="link6_flange"/>
       <child link="gripper_base"/>
       <xacro:insert_block name="origin"/>
