Commit message: Update arm_transmission.urdf.xacro

File: arm_transmission.urdf.xacro (robot description, xacro)
@@ -7,5 +7,5 @@
             </hardware>
             <joint name="link1_to_link2">
-                <command_interface name="position">
+                <command_interface name="velocity">
                     <param name="min">-2.879793</param>
                     <param name="max">2.879793</param>
@@ -15,5 +15,5 @@
             </joint>
             <joint name="link2_to_link3">
-                <command_interface name="position">
+                <command_interface name="velocity">
                     <param name="min">-2.879793</param>
                     <param name="max">2.879793</param>
@@ -23,5 +23,5 @@
             </joint>
             <joint name="link3_to_link4">
-                <command_interface name="position">
+                <command_interface name="velocity">
                     <param name="min">-2.879793</param>
                     <param name="max">2.879793</param>
@@ -31,5 +31,5 @@
             </joint>
             <joint name="link4_to_link5">
-                <command_interface name="position">
+                <command_interface name="velocity">
                     <param name="min">-2.879793</param>
                     <param name="max">2.879793</param>
@@ -39,5 +39,5 @@
             </joint>
             <joint name="link5_to_link6">
-                <command_interface name="position">
+                <command_interface name="velocity">
                     <param name="min">-2.879793</param>
                     <param name="max">2.879793</param>
@@ -47,5 +47,5 @@
             </joint>
             <joint name="link6_to_${flange_link}">
-                <command_interface name="position">
+                <command_interface name="velocity">
                     <param name="min">-3.05</param>
                     <param name="max">3.05</param>
@@ -54,5 +54,98 @@
                 <state_interface name="velocity"/>
             </joint>
+            <joint name="gripper_controller">
+                <command_interface name="velocity">
+                    <param name="min">-0.7</param>
+                    <param name="max">0.15</param>
+                </command_interface>
+                <state_interface name="position"/>
+                <state_interface name="velocity"/>
+            </joint>
+            <joint name="gripper_base_to_gripper_left2">
+                <param name="mimic">gripper_controller</param>
+                <param name="multiplier">1.0</param>
+                <state_interface name="position"/>
+                <state_interface name="velocity"/>
+            </joint>
+            <joint name="gripper_left3_to_gripper_left1">
+                <param name="mimic">gripper_controller</param>
+                <param name="multiplier">-1.0</param>
+                <state_interface name="position"/>
+                <state_interface name="velocity"/>
+            </joint>
+            <joint name="gripper_base_to_gripper_right3">
+                <param name="mimic">gripper_controller</param>
+                <param name="multiplier">-1.0</param>
+                <state_interface name="position"/>
+                <state_interface name="velocity"/>
+            </joint>
+            <joint name="gripper_base_to_gripper_right2">
+                <param name="mimic">gripper_controller</param>
+                <state_interface name="position"/>
+                <state_interface name="velocity"/>
+            </joint>
+            <joint name="gripper_right3_to_gripper_right1">
+                <param name="mimic">gripper_controller</param>
+                <param name="multiplier">1.0</param>
+                <state_interface name="position"/>
+                <state_interface name="velocity"/>
+            </joint>
         </ros2_control>
+        <!-- Simple transmissions for each joint (optional; useful for drivers/controllers expecting transmissions) -->
+        <!-- These use a 1:1 mechanical reduction and PositionJointInterface by default. -->
+        <transmission name="link1_to_link2_transmission" type="transmission_interface/SimpleTransmission">
+            <joint name="link1_to_link2">
+                <hardwareInterface>PositionJointInterface</hardwareInterface>
+            </joint>
+            <actuator name="motor1">
+                <mechanicalReduction>1.0</mechanicalReduction>
+                <hardwareInterface>PositionJointInterface</hardwareInterface>
+            </actuator>
+        </transmission>
+        <transmission name="link2_to_link3_transmission" type="transmission_interface/SimpleTransmission">
+            <joint name="link2_to_link3">
+                <hardwareInterface>PositionJointInterface</hardwareInterface>
+            </joint>
+            <actuator name="motor2">
+                <mechanicalReduction>1.0</mechanicalReduction>
+                <hardwareInterface>PositionJointInterface</hardwareInterface>
+            </actuator>
+        </transmission>
+        <transmission name="link3_to_link4_transmission" type="transmission_interface/SimpleTransmission">
+            <joint name="link3_to_link4">
+                <hardwareInterface>PositionJointInterface</hardwareInterface>
+            </joint>
+            <actuator name="motor3">
+                <mechanicalReduction>1.0</mechanicalReduction>
+                <hardwareInterface>PositionJointInterface</hardwareInterface>
+            </actuator>
+        </transmission>
+        <transmission name="link4_to_link5_transmission" type="transmission_interface/SimpleTransmission">
+            <joint name="link4_to_link5">
+                <hardwareInterface>PositionJointInterface</hardwareInterface>
+            </joint>
+            <actuator name="motor4">
+                <mechanicalReduction>1.0</mechanicalReduction>
+                <hardwareInterface>PositionJointInterface</hardwareInterface>
+            </actuator>
+        </transmission>
+        <transmission name="link5_to_link6_transmission" type="transmission_interface/SimpleTransmission">
+            <joint name="link5_to_link6">
+                <hardwareInterface>PositionJointInterface</hardwareInterface>
+            </joint>
+            <actuator name="motor5">
+                <mechanicalReduction>1.0</mechanicalReduction>
+                <hardwareInterface>PositionJointInterface</hardwareInterface>
+            </actuator>
+        </transmission>
+        <transmission name="link6_to_${flange_link}_transmission" type="transmission_interface/SimpleTransmission">
+            <joint name="link6_to_${flange_link}">
+                <hardwareInterface>PositionJointInterface</hardwareInterface>
+            </joint>
+            <actuator name="motor6">
+                <mechanicalReduction>1.0</mechanicalReduction>
+                <hardwareInterface>PositionJointInterface</hardwareInterface>
+            </actuator>
+        </transmission>
     </xacro:macro>
 </robot>
